File: SMD-schematics/Atmega32A.sch (KiCad schematic (older format))
At the start: 29 parts, among them J7 Conn_02x06_Odd_Even, J9 DB9_Female, SW1 SW_Push_Dual, SW2 SW_Push_Dual, SW3 SW_Push_Dual, U4 ATMEGA64M1-AU, U5 MAX232, Y2 16Mhz

Commit message: Adding DebugWIRE and modifications on ISP, UART, SPI connections
Parts:
- added J10: DebugWIRE, Pin_Headers:Pin_Header_Straight_2x03_Pitch2.54mm_SMD, symbol Conn_02x03_Odd_Even
- added J11: SPI/TXD, Pin_Headers:Pin_Header_Straight_1x03_Pitch2.54mm_SMD_Pin1Left, symbol Conn_01x03_Female
- added J12: SPI/RXD, Pin_Headers:Pin_Header_Straight_1x03_Pitch2.54mm_SMD_Pin1Left, symbol Conn_01x03_Female
- added J13: Debug/RST, Pin_Headers:Pin_Header_Straight_1x03_Pitch2.54mm_SMD_Pin1Left, symbol Conn_01x03_Female
- added J8: Conn_02x06_Odd_Even, Pin_Headers:Pin_Header_Straight_2x06_Pitch2.54mm_SMD, symbol Conn_02x06_Odd_Even
- added JP5: CAN-SPI, Pin_Headers:Pin_Header_Straight_1x02_Pitch2.54mm_SMD_Pin1Left, symbol Jumper_NO_Small
- J7: footprint (none) -> Pin_Headers:Pin_Header_Straight_2x06_Pitch2.54mm_SMD
- U4: footprint TQFP32 -> Housings_QFP:TQFP-32_7x7mm_Pitch0.8mm
Connections:
- net +5V: now also J10.2 (Pin_2)
- net AT-ADC1: now also J8.2 (Pin_2)
- net AT-ADC2: now also J8.4 (Pin_4)
- net AT-ADC3: now also J8.6 (Pin_6)
- net AT-ADC4: now also J8.8 (Pin_8)
- net AT-ADC5: now also J8.10 (Pin_10)
- net AT-MISO: now also U4.1 ((PCINT18/PSCIN2/OC1A/MISO_A)PD2), J10.1 (Pin_1); no longer U4.8 ((PCINT0/MISO/PSCOUT2A)PB0)
- net AT-MOSI: now also J10.4 (Pin_4), J11.3 (Pin_3); no longer U4.9 ((PCINT1/MOSI/PSCOUT2B)PB1)
- net AT-PB3: now also J8.7 (Pin_7)
- net AT-PB4: now also J8.9 (Pin_9)
- net AT-PC0/INT3: now also J8.1 (Pin_1)
- net AT-PC1: now also J8.3 (Pin_3); no longer J7.3 (Pin_3)
- net AT-PC7: now also J8.5 (Pin_5); no longer J7.5 (Pin_5)
- net AT-PD7: now also R16.2; no longer J7.11 (Pin_11)
- net AT-RX: now also J12.1 (Pin_1); no longer U4.12 ((PCINT20/ADC1/RXD/RXLIN/ICP1A/SCK_A)PD4)
- net AT-SCK: now also J10.3 (Pin_3), J12.3 (Pin_3); no longer U4.28 ((PCINT7/ADC4/SCK/PSCOUT0B)PB7)
- net AT-TX: now also J11.1 (Pin_1); no longer U4.2 ((PCINT19/TXD/TXLIN/OC0A/~SS~/MOSI_A)PD3)
- net GND: now also J10.6 (Pin_6)
- net ~AT-RST: now also J13.1 (Pin_1); no longer U4.31 ((PCINT24/OCD/~RESET~)PE0)
- net AT-PC2: now reaches U4.6 ((PCINT10/T0/TXCAN)PC2)
- net AT-PC2: now also J7.5 (Pin_5)
- net AT-PC3: now reaches U4.7 ((PCINT11/T1/ICP1B/RXCAN)PC3)
- net AT-PC3: now also J7.3 (Pin_3)
- net AT-PB1: now reaches J7.12 (Pin_12)
- net AT-PB1: now also J8.12 (Pin_12)
- removed net AT-PD2: R16.2, U4.1 ((PCINT18/PSCIN2/OC1A/MISO_A)PD2)
- new net AT-DW: J13.2 (Pin_2), U4.31 ((PCINT24/OCD/~RESET~)PE0)
- new net AT-RX/SCK_A: J12.2 (Pin_2), U4.12 ((PCINT20/ADC1/RXD/RXLIN/ICP1A/SCK_A)PD4)
- new net AT-TX/MOSI: J11.2 (Pin_2), JP5.2, U4.2 ((PCINT19/TXD/TXLIN/OC0A/~SS~/MOSI_A)PD3)
- new net CAN-CS: JP5.1
- new net CAN-MISO: U4.8 ((PCINT0/MISO/PSCOUT2A)PB0)
- new net CAN-MOSI: U4.9 ((PCINT1/MOSI/PSCOUT2B)PB1)
- new net CAN-SCK: U4.28 ((PCINT7/ADC4/SCK/PSCOUT0B)PB7)
- new net DW: J10.5 (Pin_5), J13.3 (Pin_3)
- no-connect marks 12 -> 13
Other:
- moved on the sheet: C11, D1, D2, R10, R11
