File: SMD-schematics/CAN_Peri.sch (KiCad schematic (older format))
At the start: 16 parts, among them J5 Screw_Terminal_01x02, J6 DB9_Female, U2 MCP2515-PDIP, U3 MCP2551-I/P, Y1 16Mhz

Commit message: Adding DebugWIRE and modifications on ISP, UART, SPI connections
Parts:
- JP4: footprint Pin_Headers:Pin_Header_Straight_1x02_Pitch2.54mm -> Pin_Headers:Pin_Header_Straight_1x02_Pitch2.54mm_SMD_Pin1Left
- U2: footprint Housings_DIP:DIP-18_W7.62mm_LongPads -> Housings_DIP:DIP-18_W8.89mm_SMDSocket_LongPads
Changed lines of the file:
@@
 F 0 "U2" H 3800 4425 50  0000 R CNN
 F 1 "MCP2515-PDIP" H 4950 4450 50  0000 R TNN
-F 2 "Housings_DIP:DIP-18_W7.62mm_LongPads" H 4200 2750 50  0001 C CIN
+F 2 "Housings_DIP:DIP-18_W8.89mm_SMDSocket_LongPads" H 4200 2750 50  0001 C CIN
 F 3 "" H 4300 2850 50  0001 C CNN
 	1    4200 3650
@@
 $EndComp
 $Comp
-L +5V #PWR14
+L +5V #PWR016
 U 1 1 59E4384B
 P 4200 2050
-F 0 "#PWR14" H 4200 1900 50  0001 C CNN
+F 0 "#PWR016" H 4200 1900 50  0001 C CNN
 F 1 "+5V" H 4200 2190 50  0000 C CNN
 F 2 "" H 4200 2050 50  0001 C CNN
@@
 $EndComp
 $Comp
-L GND #PWR16
+L GND #PWR017
 U 1 1 59E43851
 P 4400 2600
-F 0 "#PWR16" H 4400 2350 50  0001 C CNN
+F 0 "#PWR017" H 4400 2350 50  0001 C CNN
 F 1 "GND" H 4400 2450 50  0000 C CNN
 F 2 "" H 4400 2600 50  0001 C CNN
@@
 $EndComp
 $Comp
-L GND #PWR15
+L GND #PWR018
 U 1 1 59E43857
 P 4200 4750
-F 0 "#PWR15" H 4200 4500 50  0001 C CNN
+F 0 "#PWR018" H 4200 4500 50  0001 C CNN
 F 1 "GND" H 4200 4600 50  0000 C CNN
 F 2 "" H 4200 4750 50  0001 C CNN
@@
 $EndComp
 $Comp
-L GND #PWR13
+L GND #PWR019
 U 1 1 59E43873
 P 2700 3950
-F 0 "#PWR13" H 2700 3700 50  0001 C CNN
+F 0 "#PWR019" H 2700 3700 50  0001 C CNN
 F 1 "GND" H 2700 3800 50  0000 C CNN
 F 2 "" H 2700 3950 50  0001 C CNN
@@
 $EndComp
 $Comp
-L +5V #PWR18
+L +5V #PWR020
 U 1 1 59E438AE
 P 6400 3750
-F 0 "#PWR18" H 6400 3600 50  0001 C CNN
+F 0 "#PWR020" H 6400 3600 50  0001 C CNN
 F 1 "+5V" H 6400 3890 50  0000 C CNN
 F 2 "" H 6400 3750 50  0001 C CNN
@@
 NoConn ~ 5950 2600
 $Comp
-L GND #PWR20
+L GND #PWR021
 U 1 1 59E438B9
 P 6450 3150
-F 0 "#PWR20" H 6450 2900 50  0001 C CNN
+F 0 "#PWR021" H 6450 2900 50  0001 C CNN
 F 1 "GND" H 6450 3000 50  0000 C CNN
 F 2 "" H 6450 3150 50  0001 C CNN
@@
 CANL
 $Comp
-L +5V #PWR19
+L +5V #PWR022
 U 1 1 59E438D0
 P 6450 1350
-F 0 "#PWR19" H 6450 1200 50  0001 C CNN
+F 0 "#PWR022" H 6450 1200 50  0001 C CNN
 F 1 "+5V" H 6450 1490 50  0000 C CNN
 F 2 "" H 6450 1350 50  0001 C CNN
@@
 $EndComp
 $Comp
-L +5V #PWR17
+L +5V #PWR023
 U 1 1 59E57675
 P 5300 4500
-F 0 "#PWR17" H 5300 4350 50  0001 C CNN
+F 0 "#PWR023" H 5300 4350 50  0001 C CNN
 F 1 "+5V" H 5300 4640 50  0000 C CNN
 F 2 "" H 5300 4500 50  0001 C CNN
@@
 F 0 "JP4" H 7750 3630 50  0000 C CNN
 F 1 "Jumper_NO_Small" H 7760 3490 50  0000 C CNN
-F 2 "Pin_Headers:Pin_Header_Straight_1x02_Pitch2.54mm" H 7750 3550 50  0001 C CNN
+F 2 "Pin_Headers:Pin_Header_Straight_1x02_Pitch2.54mm_SMD_Pin1Left" H 7750 3550 50  0001 C CNN
 F 3 "" H 7750 3550 50  0001 C CNN
 	1    7750 3550
@@
 ~MCP-RST
 $Comp
-L GND #PWR22
+L GND #PWR024
 U 1 1 59E94CC7
 P 9100 4700
-F 0 "#PWR22" H 9100 4450 50  0001 C CNN
+F 0 "#PWR024" H 9100 4450 50  0001 C CNN
 F 1 "GND" H 9100 4550 50  0000 C CNN
 F 2 "" H 9100 4700 50  0001 C CNN
@@
 $EndComp
 $Comp
-L GND #PWR21
+L GND #PWR025
 U 1 1 59E9777D
 P 6700 1900
-F 0 "#PWR21" H 6700 1650 50  0001 C CNN
+F 0 "#PWR025" H 6700 1650 50  0001 C CNN
 F 1 "GND" H 6700 1750 50  0000 C CNN
 F 2 "" H 6700 1900 50  0001 C CNN
