File: SMD-schematics/CAN_Peri.sch (KiCad schematic (older format))
At the start: 7 parts, among them J5 Screw_Terminal_01x02, J6 DB9_Female, U3 MCP2551-I/P

Commit message: Updating Schematics: removing DB9 connectors and usart Transceiver
Parts:
- removed J6: DB9_Female, Connectors_DSub:DB9FC, symbol DB9_Female
Connections:
- net CANH: now also JP4.2; no longer R8.2
- net CANL: now also R8.1; no longer JP4.2
- net RXCAN: now also U3.4 (RXD); no longer U3.1 (TXD)
- net TXCAN: now also U3.1 (TXD); no longer U3.4 (RXD)
- net at JP4.1: now also R8.2; no longer R8.1
- no-connect marks 6 -> 1
Other:
- moved on the sheet: JP4, R8
Changed lines of the file:
@@
 NoConn ~ 5950 2600
 $Comp
-L GND #PWR034
+L GND #PWR030
 U 1 1 59E438B9
 P 6450 3150
-F 0 "#PWR034" H 6450 2900 50  0001 C CNN
+F 0 "#PWR030" H 6450 2900 50  0001 C CNN
 F 1 "GND" H 6450 3000 50  0000 C CNN
 F 2 "" H 6450 3150 50  0001 C CNN
@@
 CANL
 $Comp
-L +5V #PWR035
+L +5V #PWR031
 U 1 1 59E438D0
 P 6450 1350
-F 0 "#PWR035" H 6450 1200 50  0001 C CNN
+F 0 "#PWR031" H 6450 1200 50  0001 C CNN
 F 1 "+5V" H 6450 1490 50  0000 C CNN
 F 2 "" H 6450 1350 50  0001 C CNN
@@
 Text Label 7150 4700 0    60   ~ 0
 CANL
-Text Label 8050 3000 0    60   ~ 0
-CANH
-Text Label 8050 3800 0    60   ~ 0
-CANL
 $Comp
 L R R8
 U 1 1 59E6B871
-P 8050 3250
-F 0 "R8" V 8130 3250 50  0000 C CNN
-F 1 "120" V 8050 3250 50  0000 C CNN
-F 2 "Resistors_SMD:R_1206_HandSoldering" V 7980 3250 50  0001 C CNN
-F 3 "" H 8050 3250 50  0001 C CNN
-	1    8050 3250
+P 6350 4350
+F 0 "R8" V 6430 4350 50  0000 C CNN
+F 1 "120" V 6350 4350 50  0000 C CNN
+F 2 "Resistors_SMD:R_1206_HandSoldering" V 6280 4350 50  0001 C CNN
+F 3 "" H 6350 4350 50  0001 C CNN
+	1    6350 4350
 	-1   0    0    1
 $EndComp
@@
 L Jumper_NO_Small JP4
 U 1 1 59E6B8CF
-P 7750 3550
-F 0 "JP4" H 7750 3630 50  0000 C CNN
-F 1 "Jumper_NO_Small" H 7760 3490 50  0000 C CNN
-F 2 "Pin_Headers:Pin_Header_Straight_1x02_Pitch2.54mm" H 7750 3550 50  0001 C CNN
-F 3 "" H 7750 3550 50  0001 C CNN
-	1    7750 3550
+P 6750 4100
+F 0 "JP4" H 6750 4180 50  0000 C CNN
+F 1 "Jumper_NO_Small" H 6760 4040 50  0000 C CNN
+F 2 "Pin_Headers:Pin_Header_Straight_1x02_Pitch2.54mm" H 6750 4100 50  0001 C CNN
+F 3 "" H 6750 4100 50  0001 C CNN
+	1    6750 4100
 	0    1    1    0
 $EndComp
@@
 Text Label 9900 1050 0    60   ~ 0
 TXCAN
-$Comp
-L DB9_Female J6
-U 1 1 59E6BF36
-P 9800 4250
-F 0 "J6" H 9800 4800 50  0000 C CNN
-F 1 "DB9_Female" H 9800 3675 50  0000 C CNN
-F 2 "Connectors_DSub:DB9FC" H 9800 4250 50  0001 C CNN
-F 3 "" H 9800 4250 50  0001 C CNN
-	1    9800 4250
-	1    0    0    -1
-$EndComp
 Text HLabel 9350 900  0    60   Input ~ 0
 RXCAN
@@
 TXCAN
 $Comp
-L GND #PWR036
-U 1 1 59E94CC7
-P 9100 4700
-F 0 "#PWR036" H 9100 4450 50  0001 C CNN
-F 1 "GND" H 9100 4550 50  0000 C CNN
-F 2 "" H 9100 4700 50  0001 C CNN
-F 3 "" H 9100 4700 50  0001 C CNN
-	1    9100 4700
-	1    0    0    -1
-$EndComp
-$Comp
-L GND #PWR037
+L GND #PWR032
 U 1 1 59E9777D
 P 6700 1900
-F 0 "#PWR037" H 6700 1650 50  0001 C CNN
+F 0 "#PWR032" H 6700 1650 50  0001 C CNN
 F 1 "GND" H 6700 1750 50  0000 C CNN
 F 2 "" H 6700 1900 50  0001 C CNN
@@
 	1    0    0    -1
 $EndComp
-NoConn ~ 9500 3850
-NoConn ~ 9500 4350
-NoConn ~ 9500 4450
-NoConn ~ 9500 4550
-NoConn ~ 9500 4650
 $Comp
 L CP C6
@@
 	6950 2400 7100 2400
 Wire Wire Line
-	7150 4600 7400 4600
+	6850 4600 7400 4600
 Wire Wire Line
-	7400 4700 7150 4700
+	6750 4700 7400 4700
 Wire Wire Line
 	6950 2600 7100 2600
@@
 	6450 1350 6450 2100
 Wire Wire Line
-	7750 3450 8050 3450
+	6750 4000 6350 4000
 Wire Wire Line
-	8050 3450 8050 3400
-Wire Wire Line
-	8050 3000 8050 3100
+	6350 4500 6350 4800
 Wire Wire Line
 	9900 900  9350 900
@@
 	9350 1050 9900 1050
 Wire Wire Line
-	7850 3650 7850 4050
+	6850 4200 6850 4600
 Wire Wire Line
-	7850 4050 9500 4050
-Connection ~ 7850 3650
+	6750 4700 6750 4800
 Wire Wire Line
-	9500 4150 8450 4150
-Wire Wire Line
-	8450 4150 8450 3050
-Wire Wire Line
-	8450 3050 8050 3050
-Connection ~ 8050 3050
-Wire Wire Line
-	9500 4250 9250 4250
-Wire Wire Line
-	9250 4250 9250 4650
-Connection ~ 9250 4650
-Wire Wire Line
-	9100 4650 9400 4650
-Wire Wire Line
-	9400 3950 9500 3950
-Wire Wire Line
-	9400 4650 9400 3950
+	6750 4800 6350 4800
 Wire Wire Line
 	6700 1450 6450 1450
@@
 Wire Wire Line
 	6700 1800 6700 1900
+Text Label 5500 2300 2    60   ~ 0
+TXCAN
+Text Label 5500 2400 2    60   ~ 0
+RXCAN
 Wire Wire Line
-	9100 4650 9100 4700
-Text Label 5500 2300 2    60   ~ 0
-RXCAN
-Text Label 5500 2400 2    60   ~ 0
-TXCAN
+	6750 4200 6850 4200
 Wire Wire Line
-	7750 3650 8050 3650
-Wire Wire Line
-	8050 3650 8050 3800
+	6350 4000 6350 4200
 $EndSCHEMATC
